File: dombrick60d.kicad_pcb (KiCad board)
At the start: 2 copper layers, 147 parts, among them J1 AVR-ISP-6, SW1 SW_Push, U1 ATmega32U2-AU, U2 PRTR5V0U2X, Y1 16MHz

Commit message: sugoku ganbatta
Parts:
- moved R1 42.0 mm to (295.7, 64.5), turned to 270 degrees
- moved C4 19.2 mm to (275.2, 50.8), turned to 90 degrees
- moved C3 19.0 mm to (270.3, 49.7), turned to 90 degrees
- moved C1 18.7 mm to (285.9, 56.3)
- moved R3 17.5 mm to (291.2, 48.1), turned to 90 degrees
- moved U1 17.0 mm to (272.2, 58.9)
- moved C6 16.6 mm to (280.8, 54.9), turned to 315 degrees
- moved C5 15.1 mm to (280.9, 62.6), turned to 270 degrees
- moved Y1 15.0 mm to (285.8, 59.9), turned to 270 degrees
- moved C2 14.8 mm to (285.9, 63.2)
- moved F1 14.5 mm to (282.6, 44.7), turned to 0 degrees
- moved R2 14.1 mm to (288.7, 48.1), turned to 90 degrees
- moved R5 13.7 mm to (273.1, 74.3)
- moved R6 11.2 mm to (293.9, 56.9), turned to 90 degrees
- moved J1 11.1 mm to (291.6, 71.2)
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Connections:
- J1 pad 1: COL10 -> COL5
- J1 pad 3: COL8 -> COL6
- J1 pad 4: COL9 -> ROW2
- U1 pad 10: COL4 -> COL10
- U1 pad 11: COL5 -> COL9
- U1 pad 12: COL6 -> COL8
- U1 pad 15: COL8 -> COL6
- U1 pad 16: COL9 -> ROW2
- U1 pad 17: COL10 -> COL5
- U1 pad 18: COL11 -> COL4
- U1 pad 19: COL12 -> COL3
- U1 pad 20: COL13 -> COL2
- U1 pad 21: ROW0 -> COL1
- U1 pad 22: ROW1 -> COL0
- U1 pad 23: ROW2 -> ROW1
- U1 pad 25: ROW3 -> ROW0
- U1 pad 26: ROW4 -> COL13
- U1 pad 6: COL0 -> COL11
- U1 pad 7: COL1 -> COL12
- U1 pad 8: COL2 -> ROW4
- U1 pad 9: COL3 -> ROW3
Routing:
- net COL0: track 84.2 -> 315.8 mm, vias 0 -> 1
- net COL1: track 96.5 -> 301.6 mm, vias 0 -> 1
- net COL2: track 99.6 -> 286.1 mm, vias 0 -> 1
- net GND: track 0.00 -> 177.3 mm, vias 0 -> 8
- net COL5: track 83.5 -> 258.4 mm, vias 0 -> 3
- net COL6: track 89.9 -> 258.2 mm, vias 0 -> 4
- net COL3: track 99.6 -> 266.9 mm, vias 0 -> 1
- net COL4: track 83.2 -> 231.4 mm, vias 0 -> 1
- net COL7: track 105.3 -> 214.8 mm, vias 0 -> 1
- net COL8: track 92.5 -> 183.3 mm, vias 0 -> 1
- net ROW2: track 225.9 -> 311.8 mm, vias 0 -> 3
- net COL12: track 69.1 -> 146.3 mm, vias 0 -> 5
- net RESET: track 0.00 -> 69.2 mm, vias 0 -> 3
- net +5V: track 0.00 -> 66.0 mm, vias 0 -> 4
- net COL9: track 97.8 -> 155.5 mm
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Other:
- board outline added: 281 x 95.3 mm

Commit message: pcb haisen ok
Parts:
- moved D14 14.2 mm to (274.6, 27.8)
- moved D38 13.1 mm to (254.6, 66.4)
- moved D26 7.36 mm to (256.8, 42.9)
- moved C4 1.98 mm to (276.3, 49.1), turned to 45 degrees
- moved D27 1.55 mm to (264.7, 46.0)
- moved R6 0.63 mm to (293.9, 57.5)
- moved R4 0.52 mm to (293.8, 47.6)
- moved C1 0.38 mm to (285.9, 55.9)
- moved R5 0.38 mm to (273.4, 74.3)
- moved U2 0.25 mm to (292.5, 52.7)
Routing:
- net Net-(D27-Pad2): track 21.0 -> 30.9 mm
- net ROW0: track 322.0 -> 312.5 mm, vias 2 -> 0
- net ROW1: track 255.0 -> 263.9 mm
- net Net-(D14-Pad2): track 19.7 -> 28.2 mm
- net Net-(D26-Pad2): track 4.45 -> 12.1 mm
- net COL12: track 146.3 -> 138.6 mm, vias 5 -> 4
- net GND: track 177.3 -> 184.9 mm
- net COL5: track 258.4 -> 265.1 mm
- net +5V: track 66.0 -> 71.0 mm, vias 4 -> 5
- net Net-(D38-Pad2): track 10.5 -> 6.00 mm
- net ROW2: track 311.8 -> 307.5 mm, vias 3 -> 2
- net COL6: track 258.2 -> 261.7 mm
- net ROW3: track 338.5 -> 341.7 mm
- net RESET: track 69.2 -> 71.7 mm, vias 3 -> 2
- net Net-(R5-Pad2): track 14.4 -> 15.7 mm
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
Commit message: 2020-01-19 all ok lets production start
Parts:
- removed MX64: MX-NoLED, MX_Alps_Hybrid:MX-2U-NoLED
- added G***: LOGO, Type-C:dell, F.Cu at (165.0, 60.8)
- moved D14 24.3 mm to (298.2, 33.4)
- moved D13 16.7 mm to (279.4, 32.8)
- moved D12 3.86 mm to (260.5, 33.0)
- turned MX13 to 0 degrees
- turned MX14 to 0 degrees
Routing:
- net ROW0: track 312.5 -> 335.7 mm
- net Net-(D14-Pad2): track 28.2 -> 7.20 mm
- net COL13: track 51.4 -> 36.0 mm
- net COL12: track 138.6 -> 142.1 mm
- net Net-(D13-Pad2): track 4.84 -> 6.38 mm
- net Net-(D12-Pad2): track 5.46 -> 6.61 mm
- net RESET: track 71.7 -> 72.5 mm
- added copper zone on B.Cu, net GND
Other:
- board text added: "Dombrick60D : Dvorak Oriented 60% Keyboard dedicated to Dell"
